File: v1/v1.sch (KiCad schematic (older format))
At the start: 9 parts, among them J3 PWR, J4 RGB, U1 WeMos_D1_mini, U2 LevelShifter

Commit message: fix level converter footprint
Connections:
- no-connect marks 0 -> 18
Other:
- moved on the sheet: F_PWR1
Changed lines of the file:
@@
 L power:+5V #PWR0103
 U 1 1 5E0EEB47
-P 6900 3500
-F 0 "#PWR0103" H 6900 3350 50  0001 C CNN
-F 1 "+5V" H 6915 3673 50  0000 C CNN
-F 2 "" H 6900 3500 50  0001 C CNN
-F 3 "" H 6900 3500 50  0001 C CNN
-	1    6900 3500
+P 6800 3500
+F 0 "#PWR0103" H 6800 3350 50  0001 C CNN
+F 1 "+5V" H 6815 3673 50  0000 C CNN
+F 2 "" H 6800 3500 50  0001 C CNN
+F 3 "" H 6800 3500 50  0001 C CNN
+	1    6800 3500
 	1    0    0    -1
 $EndComp
@@
 Wire Wire Line
 	7200 4000 7200 3900
-Wire Wire Line
-	7200 3900 6900 3900
-Wire Wire Line
-	6900 3900 6900 3800
 Wire Wire Line
 	7300 4000 7300 3900
@@
 L Device:Polyfuse F_PWR1
 U 1 1 5E14E5B4
-P 6900 3650
-F 0 "F_PWR1" H 6988 3696 50  0000 L CNN
-F 1 "2A" H 6988 3605 50  0000 L CNN
-F 2 "Fuse:Fuse_1206_3216Metric" H 6950 3450 50  0001 L CNN
-F 3 "~" H 6900 3650 50  0001 C CNN
-	1    6900 3650
-	1    0    0    -1
-$EndComp
-Text Label 6900 3900 0    50   ~ 0
+P 6800 3750
+F 0 "F_PWR1" H 6888 3796 50  0000 L CNN
+F 1 "2A" H 6888 3705 50  0000 L CNN
+F 2 "Fuse:Fuse_1206_3216Metric" H 6850 3550 50  0001 L CNN
+F 3 "~" H 6800 3750 50  0001 C CNN
+	1    6800 3750
+	1    0    0    -1
+$EndComp
+Text Label 7200 4000 2    50   ~ 0
 5V_unfused
+$Comp
+L power:PWR_FLAG #FLG0101
+U 1 1 608FC6B6
+P 6750 3550
+F 0 "#FLG0101" H 6750 3625 50  0001 C CNN
+F 1 "PWR_FLAG" H 6750 3723 50  0000 C CNN
+F 2 "" H 6750 3550 50  0001 C CNN
+F 3 "~" H 6750 3550 50  0001 C CNN
+	1    6750 3550
+	0    -1   -1   0
+$EndComp
+Wire Wire Line
+	7800 3900 7650 3900
+Connection ~ 7650 3900
+NoConn ~ 6050 2200
+NoConn ~ 6050 2300
+NoConn ~ 6050 2400
+NoConn ~ 6050 2500
+NoConn ~ 6050 2600
+NoConn ~ 6050 2700
+NoConn ~ 6050 2800
+NoConn ~ 6050 2000
+NoConn ~ 6050 1900
+NoConn ~ 5250 2000
+NoConn ~ 5250 2300
+NoConn ~ 5250 2400
+NoConn ~ 7000 2650
+NoConn ~ 7000 2950
+NoConn ~ 7000 3050
+NoConn ~ 7600 3050
+NoConn ~ 7600 2950
+NoConn ~ 7600 2650
+Wire Wire Line
+	6800 3900 7200 3900
+Wire Wire Line
+	6800 3600 6800 3550
+Wire Wire Line
+	6750 3550 6800 3550
+Connection ~ 6800 3550
+Wire Wire Line
+	6800 3550 6800 3500
+$Comp
+L power:PWR_FLAG #FLG0102
+U 1 1 6129184A
+P 7800 3900
+F 0 "#FLG0102" H 7800 3975 50  0001 C CNN
+F 1 "PWR_FLAG" H 7800 4073 50  0000 C CNN
+F 2 "" H 7800 3900 50  0001 C CNN
+F 3 "~" H 7800 3900 50  0001 C CNN
+	1    7800 3900
+	-1   0    0    1
+$EndComp
 $EndSCHEMATC
